File: pcb/mrna_badge_v1.2.sch (EAGLE design)
At the start: 45 parts, among them T1 FS8205, U3 ATTINY24A-MU

Commit message: routed v1.2
Parts:
- U3: value ATTINY24A-MU -> ATTINY24A-MUFOOT; device Atmel_By_element14_Batch_1-00:ATTINY24A-MU -> Atmel_By_element14_Batch_1-00:ATTINY24A-MUFOOT
Changed lines of the file:
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@@
 <part name="+3V8" library="supply1" deviceset="+3V3" device=""/>
 <part name="+3V9" library="supply1" deviceset="+3V3" device=""/>
-<part name="U3" library="Atmel_By_element14_Batch_1-00" deviceset="ATTINY24A-MU" device=""/>
+<part name="U3" library="Atmel_By_element14_Batch_1-00" deviceset="ATTINY24A-MU" device="FOOT" value="ATTINY24A-MUFOOT"/>
 <part name="GND7" library="supply1" deviceset="GND" device=""/>
 <part name="3V1" library="supply1" deviceset="+3V3" device=""/>

Commit message: fixed routing issues for v1.2
Parts:
- !RES, GND, MISO, MOSI, SCK, V+: value PTR1TP15R -> (none); device testpad:PTR1TP15R -> pinhead:0.7MM_POGO-PINSPADS
- S1: device switch:TS-1088 -> switch:TS-1088NOHOLES
Connections:
- net !RES: now also !RES.1; no longer !RES.TP
- net 3V3: now also V+.1; no longer V+.TP
- net GND: now also GND.1; no longer GND.TP
- net RE1: now also MOSI.1; no longer MOSI.TP
- net YE1: now also SCK.1; no longer SCK.TP
- net YE2: now also MISO.1; no longer MISO.TP
Other:
- moved on the sheet: C4
Changed lines of the file:
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@@
 <part name="P+6" library="supply1" deviceset="+5V" device=""/>
 <part name="GND10" library="supply1" deviceset="GND" device=""/>
-<part name="S1" library="switch" deviceset="TS-1088" device=""/>
+<part name="S1" library="switch" deviceset="TS-1088" device="NOHOLES"/>
 <part name="GND9" library="supply1" deviceset="GND" device=""/>
 <part name="FRAME1" library="frames" deviceset="A4L-LOC" device=""/>
@@
 <part name="+3V11" library="supply1" deviceset="+3V3" device=""/>
 <part name="GND8" library="supply1" deviceset="GND" device=""/>
-<part name="V+" library="testpad" deviceset="PTR1" device="TP15R"/>
-<part name="!RES" library="testpad" deviceset="PTR1" device="TP15R"/>
-<part name="MOSI" library="testpad" deviceset="PTR1" device="TP15R"/>
-<part name="MISO" library="testpad" deviceset="PTR1" device="TP15R"/>
-<part name="SCK" library="testpad" deviceset="PTR1" device="TP15R"/>
-<part name="GND" library="testpad" deviceset="PTR1" device="TP15R"/>
 <part name="C4" library="rcl" deviceset="C-EU" device="C0402K" value="100n"/>
 <part name="GND11" library="supply1" deviceset="GND" device=""/>
+<part name="V+" library="pinhead" deviceset="0.7MM_POGO-PINS" device="PADS"/>
+<part name="!RES" library="pinhead" deviceset="0.7MM_POGO-PINS" device="PADS"/>
+<part name="MOSI" library="pinhead" deviceset="0.7MM_POGO-PINS" device="PADS"/>
+<part name="MISO" library="pinhead" deviceset="0.7MM_POGO-PINS" device="PADS"/>
+<part name="SCK" library="pinhead" deviceset="0.7MM_POGO-PINS" device="PADS"/>
+<part name="GND" library="pinhead" deviceset="0.7MM_POGO-PINS" device="PADS"/>
 </parts>
 <sheets>
@@
 <instance part="U3" gate="A" x="73.66" y="45.72"/>
 <instance part="GND7" gate="1" x="50.8" y="15.24" rot="MR0"/>
-<instance part="3V1" gate="G$1" x="40.64" y="76.2"/>
+<instance part="3V1" gate="G$1" x="30.48" y="73.66"/>
 <instance part="R17" gate="G$1" x="96.52" y="53.34" rot="R90"/>
 <instance part="+3V2" gate="G$1" x="96.52" y="60.96"/>
@@
 <instance part="+3V11" gate="G$1" x="198.12" y="76.2"/>
 <instance part="GND8" gate="1" x="198.12" y="53.34" rot="MR0"/>
-<instance part="V+" gate="G$1" x="205.74" y="71.12" smashed="yes" rot="R90">
-<attribute name="NAME" x="212.09" y="69.596" size="1.778" layer="95"/>
-<attribute name="TP_SIGNAL_NAME" x="208.28" y="72.39" size="1.778" layer="97" rot="R90"/>
-</instance>
-<instance part="!RES" gate="G$1" x="205.74" y="68.58" smashed="yes" rot="R90">
-<attribute name="NAME" x="212.09" y="67.056" size="1.778" layer="95"/>
-<attribute name="TP_SIGNAL_NAME" x="208.28" y="69.85" size="1.778" layer="97" rot="R90"/>
-</instance>
-<instance part="MOSI" gate="G$1" x="205.74" y="66.04" smashed="yes" rot="R90">
-<attribute name="NAME" x="212.09" y="64.516" size="1.778" layer="95"/>
-<attribute name="TP_SIGNAL_NAME" x="208.28" y="67.31" size="1.778" layer="97" rot="R90"/>
-</instance>
-<instance part="MISO" gate="G$1" x="205.74" y="63.5" smashed="yes" rot="R90">
-<attribute name="NAME" x="212.09" y="61.976" size="1.778" layer="95"/>
-<attribute name="TP_SIGNAL_NAME" x="208.28" y="64.77" size="1.778" layer="97" rot="R90"/>
-</instance>
-<instance part="SCK" gate="G$1" x="205.74" y="60.96" smashed="yes" rot="R90">
-<attribute name="NAME" x="212.09" y="59.436" size="1.778" layer="95"/>
-<attribute name="TP_SIGNAL_NAME" x="208.28" y="62.23" size="1.778" layer="97" rot="R90"/>
-</instance>
-<instance part="GND" gate="G$1" x="205.74" y="58.42" smashed="yes" rot="R90">
-<attribute name="NAME" x="212.09" y="56.896" size="1.778" layer="95"/>
-<attribute name="TP_SIGNAL_NAME" x="208.28" y="59.69" size="1.778" layer="97" rot="R90"/>
-</instance>
-<instance part="C4" gate="G$1" x="38.1" y="68.58" rot="R270"/>
-<instance part="GND11" gate="1" x="30.48" y="68.58" rot="MR90"/>
+<instance part="C4" gate="G$1" x="30.48" y="66.04"/>
+<instance part="GND11" gate="1" x="30.48" y="58.42" rot="MR0"/>
+<instance part="V+" gate="G$1" x="205.74" y="71.12"/>
+<instance part="!RES" gate="G$1" x="205.74" y="68.58"/>
+<instance part="MOSI" gate="G$1" x="205.74" y="66.04"/>
+<instance part="MISO" gate="G$1" x="205.74" y="63.5"/>
+<instance part="SCK" gate="G$1" x="205.74" y="60.96"/>
+<instance part="GND" gate="G$1" x="205.74" y="58.42"/>
 </instances>
 <busses>
@@
 <pinref part="GND8" gate="1" pin="GND"/>
 <wire x1="198.12" y1="55.88" x2="198.12" y2="58.42" width="0.1524" layer="91"/>
-<pinref part="GND" gate="G$1" pin="TP"/>
+<pinref part="GND" gate="G$1" pin="1"/>
 </segment>
 <segment>
@@
 <pinref part="U3" gate="A" pin="VCC"/>
 <pinref part="3V1" gate="G$1" pin="+3V3"/>
-<wire x1="40.64" y1="68.58" x2="40.64" y2="73.66" width="0.1524" layer="91"/>
+<wire x1="30.48" y1="68.58" x2="30.48" y2="71.12" width="0.1524" layer="91"/>
 <pinref part="C4" gate="G$1" pin="1"/>
-<junction x="40.64" y="68.58"/>
-<wire x1="40.64" y1="68.58" x2="55.88" y2="68.58" width="0.1524" layer="91"/>
+<junction x="30.48" y="68.58"/>
+<wire x1="30.48" y1="68.58" x2="55.88" y2="68.58" width="0.1524" layer="91"/>
 </segment>
 <segment>
@@
 <pinref part="+3V11" gate="G$1" pin="+3V3"/>
 <wire x1="198.12" y1="71.12" x2="198.12" y2="73.66" width="0.1524" layer="91"/>
-<pinref part="V+" gate="G$1" pin="TP"/>
+<pinref part="V+" gate="G$1" pin="1"/>
 </segment>
 </net>
@@
 <wire x1="203.2" y1="60.96" x2="198.12" y2="60.96" width="0.1524" layer="91"/>
 <label x="193.04" y="60.96" size="1.778" layer="95"/>
-<pinref part="SCK" gate="G$1" pin="TP"/>
+<pinref part="SCK" gate="G$1" pin="1"/>
 </segment>
 </net>
@@
 <wire x1="198.12" y1="63.5" x2="203.2" y2="63.5" width="0.1524" layer="91"/>
 <label x="193.04" y="63.5" size="1.778" layer="95"/>
-<pinref part="MISO" gate="G$1" pin="TP"/>
+<pinref part="MISO" gate="G$1" pin="1"/>
 </segment>
 </net>
@@
 <wire x1="203.2" y1="66.04" x2="198.12" y2="66.04" width="0.1524" layer="91"/>
 <label x="193.04" y="66.04" size="1.778" layer="95"/>
-<pinref part="MOSI" gate="G$1" pin="TP"/>
+<pinref part="MOSI" gate="G$1" pin="1"/>
 </segment>
 </net>
@@
 <wire x1="198.12" y1="68.58" x2="203.2" y2="68.58" width="0.1524" layer="91"/>
 <label x="193.04" y="68.58" size="1.778" layer="95"/>
-<pinref part="!RES" gate="G$1" pin="TP"/>
+<pinref part="!RES" gate="G$1" pin="1"/>
 </segment>
 <segment>
@@
 <wire x1="96.52" y1="48.26" x2="91.44" y2="48.26" width="0.1524" layer="91"/>
 <wire x1="91.44" y1="48.26" x2="91.44" y2="60.96" width="0.1524" layer="91"/>
-<label x="93.98" y="40.64" size="1.778" layer="95"/>
 <wire x1="91.44" y1="48.26" x2="91.44" y2="40.64" width="0.1524" layer="91"/>
 <junction x="91.44" y="48.26"/>

Commit message: patches from v1.2 fixed for v1.3
Changed lines of the file:
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@@
 <grid distance="0.1" unitdist="inch" unit="inch" style="lines" multiple="1" display="no" altdistance="0.01" altunitdist="inch" altunit="inch"/>
 <layers>
-<layer number="1" name="Top" color="4" fill="1" visible="yes" active="no"/>
-<layer number="2" name="Route2" color="16" fill="1" visible="yes" active="no"/>
-<layer number="3" name="Route3" color="17" fill="1" visible="yes" active="no"/>
-<layer number="4" name="Route4" color="18" fill="1" visible="yes" active="no"/>
-<layer number="5" name="Route5" color="19" fill="1" visible="yes" active="no"/>
-<layer number="6" name="Route6" color="25" fill="1" visible="yes" active="no"/>
-<layer number="7" name="Route7" color="26" fill="1" visible="yes" active="no"/>
-<layer number="8" name="Route8" color="27" fill="1" visible="yes" active="no"/>
-<layer number="9" name="Route9" color="28" fill="1" visible="yes" active="no"/>
-<layer number="10" name="Route10" color="29" fill="1" visible="yes" active="no"/>
-<layer number="11" name="Route11" color="30" fill="1" visible="yes" active="no"/>
-<layer number="12" name="Route12" color="20" fill="1" visible="yes" active="no"/>
-<layer number="13" name="Route13" color="21" fill="1" visible="yes" active="no"/>
-<layer number="14" name="Route14" color="22" fill="1" visible="yes" active="no"/>
-<layer number="15" name="Route15" color="23" fill="1" visible="yes" active="no"/>
-<layer number="16" name="Bottom" color="1" fill="1" visible="yes" active="no"/>
-<layer number="17" name="Pads" color="2" fill="1" visible="yes" active="no"/>
-<layer number="18" name="Vias" color="2" fill="1" visible="yes" active="no"/>
-<layer number="19" name="Unrouted" color="6" fill="1" visible="yes" active="no"/>
-<layer number="20" name="Dimension" color="24" fill="1" visible="yes" active="no"/>
-<layer number="21" name="tPlace" color="7" fill="1" visible="yes" active="no"/>
-<layer number="22" name="bPlace" color="7" fill="1" visible="yes" active="no"/>
-<layer number="23" name="tOrigins" color="15" fill="1" visible="yes" active="no"/>
-<layer number="24" name="bOrigins" color="15" fill="1" visible="yes" active="no"/>
-<layer number="25" name="tNames" color="7" fill="1" visible="yes" active="no"/>
-<layer number="26" name="bNames" color="7" fill="1" visible="yes" active="no"/>
-<layer number="27" name="tValues" color="7" fill="1" visible="yes" active="no"/>
-<layer number="28" name="bValues" color="7" fill="1" visible="yes" active="no"/>
+<layer number="1" name="Top" color="4" fill="1" visible="no" active="no"/>
+<layer number="2" name="Route2" color="16" fill="1" visible="no" active="no"/>
+<layer number="3" name="Route3" color="17" fill="1" visible="no" active="no"/>
+<layer number="4" name="Route4" color="18" fill="1" visible="no" active="no"/>
+<layer number="5" name="Route5" color="19" fill="1" visible="no" active="no"/>
+<layer number="6" name="Route6" color="25" fill="1" visible="no" active="no"/>
+<layer number="7" name="Route7" color="26" fill="1" visible="no" active="no"/>
+<layer number="8" name="Route8" color="27" fill="1" visible="no" active="no"/>
+<layer number="9" name="Route9" color="28" fill="1" visible="no" active="no"/>
+<layer number="10" name="Route10" color="29" fill="1" visible="no" active="no"/>
+<layer number="11" name="Route11" color="30" fill="1" visible="no" active="no"/>
+<layer number="12" name="Route12" color="20" fill="1" visible="no" active="no"/>
+<layer number="13" name="Route13" color="21" fill="1" visible="no" active="no"/>
+<layer number="14" name="Route14" color="22" fill="1" visible="no" active="no"/>
+<layer number="15" name="Route15" color="23" fill="1" visible="no" active="no"/>
+<layer number="16" name="Bottom" color="1" fill="1" visible="no" active="no"/>
+<layer number="17" name="Pads" color="2" fill="1" visible="no" active="no"/>
+<layer number="18" name="Vias" color="2" fill="1" visible="no" active="no"/>
+<layer number="19" name="Unrouted" color="6" fill="1" visible="no" active="no"/>
+<layer number="20" name="Dimension" color="24" fill="1" visible="no" active="no"/>
+<layer number="21" name="tPlace" color="7" fill="1" visible="no" active="no"/>
+<layer number="22" name="bPlace" color="7" fill="1" visible="no" active="no"/>
+<layer number="23" name="tOrigins" color="15" fill="1" visible="no" active="no"/>
+<layer number="24" name="bOrigins" color="15" fill="1" visible="no" active="no"/>
+<layer number="25" name="tNames" color="7" fill="1" visible="no" active="no"/>
+<layer number="26" name="bNames" color="7" fill="1" visible="no" active="no"/>
+<layer number="27" name="tValues" color="7" fill="1" visible="no" active="no"/>
+<layer number="28" name="bValues" color="7" fill="1" visible="no" active="no"/>
 <layer number="29" name="tStop" color="7" fill="3" visible="no" active="no"/>
 <layer number="30" name="bStop" color="7" fill="6" visible="no" active="no"/>
@@
 <layer number="35" name="tGlue" color="7" fill="4" visible="no" active="no"/>
 <layer number="36" name="bGlue" color="7" fill="5" visible="no" active="no"/>
-<layer number="37" name="tTest" color="7" fill="1" visible="yes" active="no"/>
-<layer number="38" name="bTest" color="7" fill="1" visible="yes" active="no"/>
+<layer number="37" name="tTest" color="7" fill="1" visible="no" active="no"/>
+<layer number="38" name="bTest" color="7" fill="1" visible="no" active="no"/>
 <layer number="39" name="tKeepout" color="4" fill="11" visible="no" active="no"/>
 <layer number="40" name="bKeepout" color="1" fill="11" visible="no" active="no"/>
@@
 <layer number="44" name="Drills" color="7" fill="1" visible="no" active="no"/>
 <layer number="45" name="Holes" color="7" fill="1" visible="no" active="no"/>
-<layer number="46" name="Milling" color="3" fill="1" visible="yes" active="no"/>
-<layer number="47" name="Measures" color="7" fill="1" visible="yes" active="no"/>
-<layer number="48" name="Document" color="7" fill="1" visible="yes" active="no"/>
-<layer number="49" name="Reference" color="7" fill="1" visible="yes" active="no"/>
-<layer number="50" name="dxf" color="7" fill="1" visible="yes" active="no"/>
-<layer number="51" name="tDocu" color="7" fill="1" visible="yes" active="no"/>
-<layer number="52" name="bDocu" color="7" fill="1" visible="yes" active="no"/>
-<layer number="53" name="tGND_GNDA" color="7" fill="9" visible="yes" active="no"/>
-<layer number="54" name="bGND_GNDA" color="7" fill="9" visible="yes" active="no"/>
-<layer number="56" name="wert" color="7" fill="1" visible="yes" active="no"/>
-<layer number="57" name="tCAD" color="7" fill="1" visible="yes" active="no"/>
-<layer number="59" name="tCarbon" color="7" fill="1" visible="yes" active="no"/>
-<layer number="60" name="bCarbon" color="7" fill="1" visible="yes" active="no"/>
+<layer number="46" name="Milling" color="3" fill="1" visible="no" active="no"/>
+<layer number="47" name="Measures" color="7" fill="1" visible="no" active="no"/>
+<layer number="48" name="Document" color="7" fill="1" visible="no" active="no"/>
+<layer number="49" name="Reference" color="7" fill="1" visible="no" active="no"/>
+<layer number="50" name="dxf" color="7" fill="1" visible="no" active="no"/>
+<layer number="51" name="tDocu" color="7" fill="1" visible="no" active="no"/>
+<layer number="52" name="bDocu" color="7" fill="1" visible="no" active="no"/>
+<layer number="53" name="tGND_GNDA" color="7" fill="9" visible="no" active="no"/>
+<layer number="54" name="bGND_GNDA" color="7" fill="9" visible="no" active="no"/>
+<layer number="56" name="wert" color="7" fill="1" visible="no" active="no"/>
+<layer number="57" name="tCAD" color="7" fill="1" visible="no" active="no"/>
+<layer number="59" name="tCarbon" color="7" fill="1" visible="no" active="no"/>
+<layer number="60" name="bCarbon" color="7" fill="1" visible="no" active="no"/>
 <layer number="88" name="SimResults" color="9" fill="1" visible="yes" active="yes"/>
 <layer number="89" name="SimProbes" color="9" fill="1" visible="yes" active="yes"/>
@@
 <wire x1="91.44" y1="48.26" x2="91.44" y2="40.64" width="0.1524" layer="91"/>
 <junction x="91.44" y="48.26"/>
-</segment>
-</net>
+<label x="91.44" y="40.64" size="1.778" layer="95"/>
+</segment>
+</net>
